File: electrical/mec-arm-esc/powerstage.kicad_sch (KiCad schematic)
At the start: 0 parts

Commit message: first half bridge added
Parts:
- added C1, C2, C3, C4: C, symbol Device:C
- added D1: D, symbol Device:D
- added Q1, Q2: STL110N10F7, EasyEDA:DFN-8_L5.8-W4.9-P1.27-LS6.0-BL-1, symbol core:STL110N10F7
- added R1, R2, R3, R4: R, symbol Device:R
- added U1: L6387ED, EasyEDA:SOIC-8_L4.9-W3.9-P1.27-LS6.0-BL, symbol core:L6387ED
Connections:
- new net: C4.1, D1.1 (K), U1.8 (VBOOT)
- new net: C1.1, U1.1 (LIN)
- new net: C2.1, U1.2 (HIN)
- new net +12V: C3.1, D1.2 (A), U1.3 (VCC)
- new net GND: C1.2, C2.2, C3.2, U1.4 (GND)
