File: electrical/mec-arm-esc/powerstage.kicad_sch (KiCad schematic)
At the start: 19 parts, among them Q1 STL110N10F7, Q2 STL110N10F7, U1 L6387ED

Commit message: added backups
Parts:
- R7: value 655 -> 518
Other:
- note added: "Current Sense Circuit sim for internal MCU Opamp. For this esc, the internal opamps in the motor driver will be leveraged in an effort to save on signal integrity, as it is differential pairs compared to the signle eded opamps offered directly on the stm32. Internal Opamp can only amplify with gains of 5, 10, 20, and 40. Thus, this had to be taken into consideration when sizing the shunt resistor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"
- note removed: "Current Sense Circuit sim for internal MCU Opamp. For this esc, the internal opamps in the MCu will be leveraged in an effort to save on routing space, and costs. Internal Opamp can only amplify with gains with powers of 2, so this had to be takeninto consideration when sizing the shunt resistor, along with resolution adn power constrainrs. A 4m resistor was selected in order to maximize the tota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"

Commit message: Finished Bare MCU + Oscillator, added prelim powerstage additions
Parts:
- added R10: SEWF3920D4L00P9, EasyEDA:RES-SMD_L10.0-W5.2-1, symbol core:SEWF3920D4L00P9
- added U3: DRV8323SRTAT, EasyEDA:WQFN-40_L6.0-W6.0-P0.50-TL-EP4.5, symbol core:DRV8323SRTAT
Connections:
- net GND: now also R10.1, U3.10 (SNA)
- net PHASE A: no longer Q1.1 (S), Q1.2 (S), Q1.3 (S), Q2.5 (D), Q2.6 (D), Q2.7 (D), Q2.8 (D), Q2.9 (D)
- net VBUS: no longer Q1.5 (D), Q1.6 (D), Q1.7 (D), Q1.8 (D), Q1.9 (D)
- net V_SHUNT_A+: no longer Q2.1 (S), Q2.2 (S), Q2.3 (S)
- net at R2.1, R4.2: no longer Q2.4 (G)
- net at R1.2, R3.2: no longer Q1.4 (G)
- new net: Q2.1 (S), Q2.2 (S), Q2.3 (S), R10.2, U3.9 (SPA)
- new net: Q1.1 (S), Q2.6 (D)
- new net: Q1.2 (S), Q2.7 (D)
- new net: Q1.3 (S), Q2.8 (D)
- new net: Q2.4 (G), U3.8 (GLA)
- new net GHA: Q1.4 (G), U3.6 (GHA)
- new net PHASE_A: Q2.5 (D), Q2.9 (D), U3.7 (SHA)
- new net VDRAIN: U3.5 (VDRAIN)
- new net VM: U3.4 (VM)
Other:
- note added: "Current Sense Discussion For this esc setup, the motor driver ensures that VREF/2 is the middle reference point for the current sensing, where here VREF is 3V3. From here, a gain of 10 is selected, in order to provide the mcu with an idle voltage of 1.65V when there is no current flowing through a phase. This means, that under peak load (22A), we can expect a max voltage (assuming 4m shunt) of: V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"
- note removed: "Current Sense Circuit sim for internal MCU Opamp. For this esc, the internal opamps in the motor driver will be leveraged in an effort to save on signal integrity, as it is differential pairs compared to the signle eded opamps offered directly on the stm32. Internal Opamp can only amplify with gains of 5, 10, 20, and 40. Thus, this had to be taken into consideration when sizing the shunt resistor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"

Commit message: Completed inverter, started calculation for input power
Parts:
- removed C1, C2: 100pF, symbol Device:C
- removed C3: 470nF, symbol Device:C
- removed C4: 1uF, symbol Device:C
- removed C5: 10nF, symbol Device:C
- removed C6: 220 pF, symbol Device:C
- removed D2: STPS0560Z, EasyEDA:SOD-123_L2.7-W1.6-LS3.7-RD, symbol core:STPS0560Z
- removed R1, R2: 10k, symbol Device:R
- removed R3, R4: 33, symbol Device:R
- removed R5: 1, symbol Device:R
- removed R6: SEWF3920D4L00P9, EasyEDA:RES-SMD_L10.0-W5.2-1, symbol core:SEWF3920D4L00P9
- removed R7: 518, symbol Device:R
- removed R8, R9: 22k, symbol Device:R
- removed U1: L6387ED, EasyEDA:SOIC-8_L4.9-W3.9-P1.27-LS6.0-BL, symbol core:L6387ED
- added C19, C23, C25, C26, C27: 1uF, symbol Device:C
- added C20: 47nF, symbol Device:C
- added C21, C24: 0.1uF, symbol Device:C
- added C22, C28, C29: 10uF, symbol Device:C
- added Q3, Q4, Q5, Q6: STL110N10F7, EasyEDA:DFN-8_L5.8-W4.9-P1.27-LS6.0-BL-1, symbol core:STL110N10F7
- added R12, R13: SEWF3920D4L00P9, EasyEDA:RES-SMD_L10.0-W5.2-1, symbol core:SEWF3920D4L00P9
- added R14: 0, symbol Device:R
- added R15: 10k, symbol Device:R
Connections:
- net VDRAIN is gone; now on net VBUS: U3.5 (VDRAIN)
- net VM is gone; now on net VBUS: U3.4 (VM)
- net +3V3: now also U3.24 (VREF), C24.1, R15.1
- net GND: now also U3.11 (SNB), U3.20 (SNC), U3.32 (AGND), U3.40 (PGND), U3.41 (EP), C21.2, C22.2, C23.2, C24.2, C25.2, C26.2, C27.2, C28.2, C29.2, R12.1, R13.1, R14.1
- net PHASE_A: now also Q1.1 (S), Q1.2 (S), Q1.3 (S), Q2.6 (D), Q2.7 (D), Q2.8 (D)
- net VBUS: now also Q1.5 (D), Q1.6 (D), Q1.7 (D), Q1.8 (D), Q1.9 (D), C19.1, C21.1, C22.1, C25.1, C26.1, C27.1, C28.1, C29.1, Q3.5 (D), Q3.6 (D), Q3.7 (D), Q3.8 (D), Q3.9 (D), Q5.5 (D), Q5.6 (D), Q5.7 (D), Q5.8 (D), Q5.9 (D)
- net SPA: now reaches Q2.1 (S), Q2.2 (S), Q2.3 (S), R10.2, U3.9 (SPA)
- net GLA: now reaches Q2.4 (G), U3.8 (GLA)
- net at U3.1 (CPL): now also C20.1
- net SPB: now reaches U3.12 (SPB)
- net SPB: now also Q4.1 (S), Q4.2 (S), Q4.3 (S), R12.2
- net GLB: now reaches U3.13 (GLB)
- net GLB: now also Q4.4 (G)
- net PHASE_B: now reaches U3.14 (SHB)
- net PHASE_B: now also Q3.1 (S), Q3.2 (S), Q3.3 (S), Q4.5 (D), Q4.6 (D), Q4.7 (D), Q4.8 (D), Q4.9 (D)
- net GHB: now reaches U3.15 (GHB)
- net GHB: now also Q3.4 (G)
- net GHC: now reaches U3.16 (GHC)
- net GHC: now also Q5.4 (G)
- net PHASE_C: now reaches U3.17 (SHC)
- net PHASE_C: now also Q5.1 (S), Q5.2 (S), Q5.3 (S), Q6.5 (D), Q6.6 (D), Q6.7 (D), Q6.8 (D), Q6.9 (D)
- net GLC: now reaches U3.18 (GLC)
- net GLC: now also Q6.4 (G)
- net SPC: now reaches U3.19 (SPC)
- net SPC: now also Q6.1 (S), Q6.2 (S), Q6.3 (S), R13.2
- net at U3.2 (CPH): now also C20.2
- net I_SENSE_C_ADC3: now reaches U3.21 (SOC)
- net I_SENSE_B_ADC2: now reaches U3.22 (SOB)
- net I_SENSE_A_ADC1: now reaches U3.23 (SOA)
- net DRV_nFault: now reaches U3.25 (nFAULT)
- net SPI_MISO: now reaches U3.26 (SDO)
- net SPI_MISO: now also R15.2
- net SPI_MOSI: now reaches U3.27 (SDI)
- net SPI_SCK: now reaches U3.28 (SCLK)
- net SPI_DRV_NSCS: now reaches U3.29 (nSCS)
- net VCP: now reaches U3.3 (VCP)
- net VCP: now also C19.2
- net DRV_EN: now reaches U3.30 (ENABLE)
- net at U3.31 (CAL): now also R14.2
- net at U3.33 (DVDD): now also C23.1
- net TIM1_CH1: now reaches U3.34 (INHA)
- net TIM1_CH1N: now reaches U3.35 (INLA)
- net TIM1_CH2: now reaches U3.36 (INHB)
- net TIM1_CH2N: now reaches U3.37 (INLB)
- net TIM1_CH3: now reaches U3.38 (INHC)
- net TIM1_CH3N: now reaches U3.39 (INLC)
Other:
- note added: "Place 1uF near high side fets"
- note added: "This capacitor bank is expected to handle a total ripple current of: i_c = 0.65 * I_phase_rms * 1.1 = 0.65 * 15.56 *1.1 = 11.12A The total amount of capacitance required for full load would be: C = i_c /(delta_V * f_sw). Given a 10% maximum allowable voltage ripple on the DC Bus, the require capacitance is: C = 11.12 / (2.4 * 25k) = 185uF Taking a 10uF capacitor, we will need 18 caps."
- moved on the sheet: Q1, Q2, R10, U3

Commit message: Changed the components in all the drawings to reflect the new library, and added vbus sensing
Parts:
- removed R10, R12, R13: SEWF3920D4L00P9, EasyEDA:RES-SMD_L10.0-W5.2-1, symbol core:SEWF3920D4L00P9
- added C30: 15uF, Capacitor_SMD:C_0805_2012Metric, symbol Device:C
- added C31, C32, C33, C34, C35, C36, C37, C38, C39, C40, C41: 15uF, symbol Device:C
- added R1, R2, R3: SEWF3920D4L00P9, core:RES-SMD_L10.0-W5.2-1, symbol core:SEWF3920D4L00P9
- Q1, Q2, Q3, Q4, Q5, Q6: footprint EasyEDA:DFN-8_L5.8-W4.9-P1.27-LS6.0-BL-1 -> core:DFN-8_L5.8-W4.9-P1.27-LS6.0-BL-1
- U3: footprint EasyEDA:WQFN-40_L6.0-W6.0-P0.50-TL-EP4.5 -> core:WQFN-40_L6.0-W6.0-P0.50-TL-EP4.5
Connections:
- net +3V3: now also U3.17 (SHC); no longer U3.24 (VREF)
- net DRV_EN: now also U3.11 (SNB); no longer U3.30 (ENABLE)
- net DRV_nFault: now also U3.16 (GHC); no longer U3.25 (nFAULT)
- net GHA: now also U3.35 (INLA); no longer U3.6 (GHA)
- net GHB: now also U3.30 (ENABLE); no longer U3.15 (GHB)
- net GHC: now also U3.25 (nFAULT); no longer U3.16 (GHC)
- net GLA: now also U3.33 (DVDD); no longer U3.8 (GLA)
- net GLB: now also U3.28 (SCLK); no longer U3.13 (GLB)
- net GLC: now also U3.23 (SOA); no longer U3.18 (GLC)
- net GND: now also U3.1 (CPL), U3.21 (SOC), U3.26 (SDO), U3.31 (CAL), U3.9 (SPA), C30.2, C31.2, C32.2, C33.2, C34.2, C35.2, C36.2, C37.2, C38.2, C39.2, C40.2, C41.2, R1.1, R2.1, R3.1; no longer U3.10 (SNA), U3.11 (SNB), U3.20 (SNC), U3.32 (AGND), U3.40 (PGND)
- net I_SENSE_A_ADC1: now also U3.18 (GLC); no longer U3.23 (SOA)
- net I_SENSE_B_ADC2: now also U3.19 (SPC); no longer U3.22 (SOB)
- net I_SENSE_C_ADC3: now also U3.20 (SNC); no longer U3.21 (SOC)
- net PHASE_A: now also U3.34 (INHA); no longer U3.7 (SHA)
- net PHASE_B: now also U3.29 (nSCS); no longer U3.14 (SHB)
- net PHASE_C: now also U3.24 (VREF); no longer U3.17 (SHC)
- net SPA: now also U3.32 (AGND), R1.2; no longer U3.9 (SPA)
- net SPB: now also U3.27 (SDI), R2.2; no longer U3.12 (SPB)
- net SPC: now also U3.22 (SOB), R3.2; no longer U3.19 (SPC)
- net SPI_DRV_NSCS: now also U3.12 (SPB); no longer U3.29 (nSCS)
- net SPI_MISO: now also U3.15 (GHB); no longer U3.26 (SDO)
- net SPI_MOSI: now also U3.14 (SHB); no longer U3.27 (SDI)
- net SPI_SCK: now also U3.13 (GLB); no longer U3.28 (SCLK)
- net TIM1_CH1: now also U3.7 (SHA); no longer U3.34 (INHA)
- net TIM1_CH1N: now also U3.6 (GHA); no longer U3.35 (INLA)
- net TIM1_CH2: now also U3.5 (VDRAIN); no longer U3.36 (INHB)
- net TIM1_CH2N: now also U3.4 (VM); no longer U3.37 (INLB)
- net TIM1_CH3: now also U3.3 (VCP); no longer U3.38 (INHC)
- net TIM1_CH3N: now also U3.2 (CPH); no longer U3.39 (INLC)
- net VBUS: now also U3.36 (INHB), U3.37 (INLB), C30.1, C31.1, C32.1, C33.1, C34.1, C35.1, C36.1, C37.1, C38.1, C39.1, C40.1, C41.1; no longer U3.4 (VM), U3.5 (VDRAIN)
- net VCP: now also U3.38 (INHC); no longer U3.3 (VCP)
- net at R14.2: now also U3.10 (SNA); no longer U3.31 (CAL)
- net at C20.1: now also U3.40 (PGND); no longer U3.1 (CPL)
- net at C20.2: now also U3.39 (INLC); no longer U3.2 (CPH)
- net at C23.1: now also U3.8 (GLA); no longer U3.33 (DVDD)
Other:
- note added: "These are not going to be assembled, already have in stock"
- note added: "This capacitor bank is expected to handle a total ripple current of: i_c = 0.65 * I_phase_rms * 1.1 = 0.65 * 15.56 *1.1 = 11.12A The total amount of capacitance required for full load would be: C = i_c /(delta_V * f_sw). Given a 10% maximum allowable voltage ripple on the DC Bus, the require capacitance is: C = 11.12 / (2.4 * 25k) = 185uF Taking a 15uF capacitor, we will need 12 caps, each capabl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"
- note removed: "This capacitor bank is expected to handle a total ripple current of: i_c = 0.65 * I_phase_rms * 1.1 = 0.65 * 15.56 *1.1 = 11.12A The total amount of capacitance required for full load would be: C = i_c /(delta_V * f_sw). Given a 10% maximum allowable voltage ripple on the DC Bus, the require capacitance is: C = 11.12 / (2.4 * 25k) = 185uF Taking a 10uF capacitor, we will need 18 caps."
