File: electrical/mec-arm-esc/powerstage.kicad_sch (KiCad schematic)
At the start: 35 parts, among them Q1 STL110N10F7, Q2 STL110N10F7, Q3 STL110N10F7, Q4 STL110N10F7, Q5 STL110N10F7, Q6 STL110N10F7, U3 DRV8323SRTAT

Commit message: Schematic Done, review 1
Parts:
- added C49: 0.47uF, symbol Device:C
- added C50, C53, C54, C58, C59, C60: 1uF, symbol Device:C
- added C51, C52: 100nF, symbol Device:C
- added C55, C56: 47uF, symbol Device:C
- added C57: 1pF, symbol Device:C
- added C61: 33uF, symbol Device:C
- added C62: 100pF, Capacitor_SMD:C_0805_2012Metric, symbol Device:C
- added C63: 2.2uF, Capacitor_SMD:C_0805_2012Metric, symbol Device:C
- added D10: SMBJ14A_C315990, core:SMB_L4.4-W3.6-LS5.4-RD, symbol core:SMBJ14A_C315990
- added D11: SMBJ30A-TR, core:SMB_L4.6-W3.6-LS5.3-RD, symbol core:SMBJ30A-TR
- added J8: Conn_01x04, Connector_PinHeader_2.54mm:PinHeader_1x04_P2.54mm_Vertical, symbol Connector_Generic:Conn_01x04
- added J9: XT30PW-M, connector:CONN-TH_XT30PW-M, symbol connector:XT30PW-M
- added L1: 15uH, core:IND-SMD_L8.0-W8.0_1217AS-H-330M, symbol core:1217AS-H-150M=P3
- added LED1, LED2, LED3, LED6: 150060RS75000, core:LED0603-RD_RED, symbol core:150060RS75000
- added Q9: STL110N10F7, core:DFN-8_L5.8-W4.9-P1.27-LS6.0-BL-1, symbol core:STL110N10F7
- added R12: 2.55M, symbol Device:R
- added R13: 200k, symbol Device:R
- added R42, R44: 100k, symbol Device:R
- added R43: 19.1k, symbol Device:R
- added R45: 40k, symbol Device:R
- added R47, R48, R55, R56, R57, R58: 1k, symbol Device:R
- added R49: 500, symbol Device:R
- added R54: 5.1k, symbol Device:R
- added R59: 10k, symbol Device:R
- added TP1, TP2, TP3, TP4: (no value), TestPoint:TestPoint_Pad_D1.5mm, symbol connector:TestPoint
- added U6: TPS2116DRLR, core:SOT-583-8_L2.1-W1.6-P0.50-LS1.6-BL, symbol core:TPS2116DRLR
- added U7: LMR51625XDDCR_C44750835, core:SOT-23-6_L2.9-W1.6-P0.95-LS2.9-BL, symbol core:LMR51625XDDCR_C44750835
- added U8: LM3940IMPX-3.3/NOPB, core:SOT-223-4_L6.5-W3.5-P2.30-LS7.0-BR, symbol core:LM3940IMPX-3.3_NOPB
- added U9: LM74610QDGKRQ1, core:VSSOP-8_L3.0-W3.0-P0.65-LS5.0-BL, symbol core:LM74610QDGKRQ1
Connections:
- net +3V3: now also U3.24 (VREF), C61.1, R49.2, R54.2, R57.2, U8.3 (OUT); no longer U3.17 (SHC)
- net DRV_EN: now also U3.30 (ENABLE); no longer U3.11 (SNB)
- net DRV_nFault: now also U3.25 (nFAULT), R54.1; no longer U3.16 (GHC)
- net GHA: now also U3.6 (GHA); no longer U3.35 (INLA)
- net GHB: now also U3.15 (GHB); no longer U3.30 (ENABLE)
- net GHC: now also U3.16 (GHC); no longer U3.25 (nFAULT)
- net GLA: now also U3.8 (GLA); no longer U3.33 (DVDD)
- net GLB: now also U3.13 (GLB); no longer U3.28 (SCLK)
- net GLC: now also U3.18 (GLC); no longer U3.23 (SOA)
- net GND: now also U3.10 (SNA), U3.11 (SNB), U3.20 (SNC), U3.32 (AGND), U3.40 (PGND), C49.2, C50.1, C52.1, C53.1, C54.1, C55.1, C56.1, C58.1, C59.2, C60.2, C61.2, C62.2, D10.1, J9.1 (-), LED1.1 (K), LED2.1 (K), LED3.1 (K), LED6.1 (K), R13.1, R43.1, R45.1, R58.2, U6.1 (GND), U7.4 (GND), U8.2 (GND), U8.4 (GND); no longer U3.1 (CPL), U3.21 (SOC), U3.26 (SDO), U3.31 (CAL), U3.9 (SPA)
- net I_SENSE_A_ADC1: now also U3.23 (SOA); no longer U3.18 (GLC)
- net I_SENSE_B_ADC2: now also U3.22 (SOB); no longer U3.19 (SPC)
- net I_SENSE_C_ADC3: now also U3.21 (SOC); no longer U3.20 (SNC)
- net PHASE_A: now also U3.7 (SHA); no longer U3.34 (INHA)
- net PHASE_B: now also U3.14 (SHB); no longer U3.29 (nSCS)
- net PHASE_C: now also U3.17 (SHC); no longer U3.24 (VREF)
- net SPA: now also U3.9 (SPA); no longer U3.32 (AGND)
- net SPB: now also U3.12 (SPB); no longer U3.27 (SDI)
- net SPC: now also U3.19 (SPC); no longer U3.22 (SOB)
- net SPI_DRV_NSCS: now also U3.29 (nSCS); no longer U3.12 (SPB)
- net SPI_MISO: now also U3.26 (SDO); no longer U3.15 (GHB)
- net SPI_MOSI: now also U3.27 (SDI); no longer U3.14 (SHB)
- net SPI_SCK: now also U3.28 (SCLK); no longer U3.13 (GLB)
- net TIM1_CH1: now also U3.34 (INHA); no longer U3.7 (SHA)
- net TIM1_CH1N: now also U3.35 (INLA); no longer U3.6 (GHA)
- net TIM1_CH2: now also U3.36 (INHB); no longer U3.5 (VDRAIN)
- net TIM1_CH2N: now also U3.37 (INLB); no longer U3.4 (VM)
- net TIM1_CH3: now also U3.38 (INHC); no longer U3.3 (VCP)
- net TIM1_CH3N: now also U3.39 (INLC); no longer U3.2 (CPH)
- net VBUS: now also U3.4 (VM), U3.5 (VDRAIN), C50.2, C52.2, C53.2, C54.2, Q9.5 (D), Q9.6 (D), Q9.7 (D), Q9.8 (D), Q9.9 (D), R12.2, R55.2, R59.2, U7.3 (VIN), U9.8 (Cathode); no longer U3.36 (INHB), U3.37 (INLB)
- net VCP: now also U3.3 (VCP); no longer U3.38 (INHC)
- net at R14.2: now also U3.31 (CAL); no longer U3.10 (SNA)
- net at C20.1: now also U3.1 (CPL); no longer U3.40 (PGND)
- net at C20.2: now also U3.2 (CPH); no longer U3.39 (INLC)
- net at C23.1: now also U3.33 (DVDD); no longer U3.8 (GLA)
- new net: C63.1, U9.1 (VCAPL)
- new net: C63.2, U9.7 (VCAPH)
- new net: C57.1, R42.1, R43.2, U7.1 (FB)
- new net: Q9.4 (G), U9.2 (Gate-PD), U9.6 (Gate-Drive)
- new net: LED1.2 (A), R47.1
- new net: D10.2, D11.2 (A)
- new net: J8.1 (Pin_1), R55.1
- new net: J8.2 (Pin_2), R56.1
- new net: J8.3 (Pin_3), R57.1
- new net: J8.4 (Pin_4), R58.1
- new net: R44.1, R45.2, U6.4 (PR1)
- new net: C51.2, L1.1, U7.5 (SW)
- new net: LED2.2 (A), R48.1
- new net: R12.1, R13.2, U7.2 (EN)
- new net: TP1.1, U6.8 (ST)
- new net: LED6.2 (A), R59.1
- new net: LED3.2 (A), R49.1
- new net: C51.1, U7.6 (CB)
- new net +5V_ESC: C49.1, C60.1, R48.2, R56.2, U6.2 (VOUT), U6.7 (VOUT), U8.1 (IN)
- new net +5V_INT: C55.2, C56.2, C57.2, C58.2, L1.2, R42.2, R44.2, R47.2, TP2.1, TP3.1, U6.3 (VIN1), U6.5 (MODE)
- new net +5V_USB: C59.1, TP4.1, U6.6 (VIN2)
- new net PWR_IN: C62.1, D11.1 (K), J9.2 (+), Q9.1 (S), Q9.2 (S), Q9.3 (S), U9.4 (Anode)
- no-connect marks 0 -> 4
Other:
- note added: "*Specific Layout Rules"
- note added: "18V UVLO Prot (thresh 0.958)"
- note added: "24V-5V Buck"
- note added: "5V - 3V3"
- note added: "5V MUX"
- note added: "DC-DC CONVERTERS + 5V MUX"
- note added: "EXPOSED POWER RAILS"
- note added: "INPUT POWER"
- note added: "INVERTER"
- note added: "Input Filter"
- note added: "Primary use case here is to measure the voltage rails, not provide power.If needed, resistors can be changed to 0 ohm"
- note added: "Reverse Polarity Protection"
- note added: "STATUS LEDS"
- note added: "These caps are not going to be assembled, already have in stock"
- note added: "This capacitor bank is expected to handle a total ripple current of: i_c = 0.65 * I_phase_rms * 1.1 = 0.65 * 15.56 *1.1 = 11.12A The total amount of capacitance required for full load would be: C = i_c /(delta_V * f_sw). Given 10% max allowable voltage ripple on the DC Bus, capacitance required is: C = 11.12 / (2.4 * 25k) = 185uF Taking a 15uF capacitor, we will need 12 caps, each capable of deli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"
- note added: "This mux selects between the 5V produced by the buck if Vbus is present, or the 5V over USB if it is connected. It puts priority on the onboard 5V produced by thebuck converter (if both are present)"
- note added: "https://webench.ti.com/appinfo/webench/scripts/SDP.cgi?ID=DCC915FA82E52C05"
- note removed: "These are not going to be assembled, already have in stock"
- note removed: "This capacitor bank is expected to handle a total ripple current of: i_c = 0.65 * I_phase_rms * 1.1 = 0.65 * 15.56 *1.1 = 11.12A The total amount of capacitance required for full load would be: C = i_c /(delta_V * f_sw). Given a 10% maximum allowable voltage ripple on the DC Bus, the require capacitance is: C = 11.12 / (2.4 * 25k) = 185uF Taking a 15uF capacitor, we will need 12 caps, each capabl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"
- moved on the sheet: C19, C20, C21, C22, C23, C24, C25, C26, C27, C28, C29, C30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

Commit message: Done placement, starting routing
Parts:
- removed C62: 100pF, Capacitor_SMD:C_0805_2012Metric, symbol Device:C
- removed C63: 2.2uF, Capacitor_SMD:C_0805_2012Metric, symbol Device:C
- removed D10: SMBJ14A_C315990, core:SMB_L4.4-W3.6-LS5.4-RD, symbol core:SMBJ14A_C315990
- removed L1: 15uH, core:IND-SMD_L8.0-W8.0_1217AS-H-330M, symbol core:1217AS-H-150M=P3
- removed Q9: STL110N10F7, core:DFN-8_L5.8-W4.9-P1.27-LS6.0-BL-1, symbol core:STL110N10F7
- removed R1, R2, R3: SEWF3920D4L00P9, core:RES-SMD_L10.0-W5.2-1, symbol core:SEWF3920D4L00P9
- removed U8: LM3940IMPX-3.3/NOPB, core:SOT-223-4_L6.5-W3.5-P2.30-LS7.0-BR, symbol core:LM3940IMPX-3.3_NOPB
- removed U9: LM74610QDGKRQ1, core:VSSOP-8_L3.0-W3.0-P0.65-LS5.0-BL, symbol core:LM74610QDGKRQ1
- added C64, C65, C66, C67, C68, C69: 10uF, core:C_0603, symbol Device:C
- added D10: 12V, core:SOD-123F_L2.8-W1.8-LS3.7-RD, symbol core:BZT52C12-13-F
- added J10: (no value), my_connector:PHASE_PAD, symbol my_connector:PHASE_PADS
- added L1: 15uH, core:IND-SMD_L6.0-W6.0_VLS6045EX, symbol core:VLS6045EX-150M
- added Q9: TJ60S04M3L-VB, core:TO-252-2_L6.6-W6.1-P4.58-LS9.9-TL, symbol core:TJ60S04M3L-VB
- added R1, R2, R3: PEWF2512D2L00Q9, core:RES-SMD_L6.3-W3.2_R2512, symbol core:PEWF2512D2L00Q9
- added R24: 10k, core:R0603, symbol Device:R
- added R62, R63, R64, R65, R66, R67: 1k, core:R_0603, symbol Device:R
- added R68: 0, core:R_0603, symbol Device:R
- added U8: AP7366EA-33W5-7, core:SOT-23-5_L3.0-W1.6-P0.95-LS2.8-BR, symbol core:AP7366EA-33W5-7
- C19, C20, C21, C22, C23, C24, C25, C26, C27, C50, C51, C52, C53, C54, C55, C56, C57, C58, C59, C60: footprint (none) -> core:C_0603
- C28, C29, C31, C32, C33, C34, C35, C36, C37, C38, C39, C40, C41: footprint (none) -> core:C_0805
- C30: footprint Capacitor_SMD:C_0805_2012Metric -> core:C_0805
- C49: value 0.47uF -> 1uF; footprint (none) -> core:C_0603
- C61: value 33uF -> 1uF; footprint (none) -> core:C_0603
- J8: now not fitted
- J9: footprint connector:CONN-TH_XT30PW-M -> my_connector:CONN-TH_XT30PW-M
- R12, R13, R14, R15, R42, R43, R44, R45, R47, R48, R49, R54, R55, R56, R57, R58, R59: footprint (none) -> core:R_0603
Connections:
- net +3V3: now also U8.5 (OUT)
- net +5V_ESC: now also U8.1 (IN), U8.3 (EN)
- net +5V_INT: now also L1.2
- net GND: now also R68.1; no longer C21.2, C22.2, C25.2, C26.2, C27.2, C28.2, C29.2, C30.2, C31.2, C32.2, C33.2, C34.2, C35.2, C36.2, C37.2, C38.2, C39.2, C40.2, C41.2, C49.2, C50.1, C52.1, C53.1, C54.1, C55.1, C56.1, C58.1, C59.2, C60.2, C61.2, J9.1 (-), LED1.1 (K), LED2.1 (K), LED3.1 (K), LED6.1 (K), R13.1, R43.1, R45.1, U3.10 (SNA), U3.11 (SNB), U3.20 (SNC), U3.40 (PGND), U3.41 (EP), U6.1 (GND), U7.4 (GND)
- net PHASE_A: now also C64.2, J10.3, R63.1
- net PHASE_B: now also C66.2, J10.2, R65.1
- net PHASE_C: now also C68.2, J10.1, R67.1
- net PWR_IN: now also Q9.2 (D); no longer D11.1 (K)
- net SPA: now also C65.2, R1.2
- net SPB: now also C67.2, R2.2
- net SPC: now also C69.2, R3.2
- net VBUS: now also D11.1 (K), D10.1 (K), Q9.3 (S), R62.1, R64.1, R66.1
- net PGND: now reaches D11.2 (A)
- net PGND: now also C21.2, C22.2, C25.2, C26.2, C27.2, C28.2, C29.2, C30.2, C31.2, C32.2, C33.2, C34.2, C35.2, C36.2, C37.2, C38.2, C39.2, C40.2, C41.2, C49.2, C50.1, C52.1, C53.1, C54.1, C55.1, C56.1, C58.1, C59.2, C60.2, C61.2, J9.1 (-), LED1.1 (K), LED2.1 (K), LED3.1 (K), LED6.1 (K), R13.1, R43.1, R45.1, U3.10 (SNA), U3.11 (SNB), U3.20 (SNC), U3.40 (PGND), U3.41 (EP), U6.1 (GND), U7.4 (GND), R1.1, R2.1, R24.1, R3.1, R68.2, U8.2 (GND)
- net at C51.2, U7.5 (SW): now also L1.1
- new net: C68.1, R66.2
- new net: C64.1, R62.2
- new net: C65.1, R63.2
- new net: C66.1, R64.2
- new net: D10.2 (A), Q9.1 (G), R24.2
- new net: C67.1, R65.2
- new net: C69.1, R67.2
- no-connect marks 4 -> 3
Other:
- note added: "25V rated"
- note added: "NET TIE"
- note added: "Phase Pads"
- note added: "This is used for Layout mostly as a ref"
- note added: "Using an Ideal Diode Controller was initially used, but replaced with a PMOS after considering regenerative affects from the motor, causing the controller to potentially shut off power"
- note added: "Values for Snubber will be experimentally determined before population"
- moved on the sheet: C30, C31, C32, C33, C34, C35, C36, C37, C38, C39, C40, C41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

Commit message: All signal routing finishes, power and planes not yet
Parts:
- removed J8: Conn_01x04, Connector_PinHeader_2.54mm:PinHeader_1x04_P2.54mm_Vertical, symbol Connector_Generic:Conn_01x04
- removed R68: 0, core:R_0603, symbol Device:R
- added J8: (no value), my_connector:TestPadArray1x4, symbol my_connector:TestPads
- C19: LCSC Part (none) -> C14664
- C20: LCSC Part (none) -> C513577
- C21, C51, C52: LCSC Part (none) -> C14663
- C22: footprint core:C_0603 -> core:C_0805; LCSC Part (none) -> C162422
- C23: value 1uF -> 1uF 6.3V; LCSC Part (none) -> C2169508
- C24: LCSC Part (none) -> C108079
- C25, C26, C27, C50, C53, C54: LCSC Part (none) -> C559769
- C28, C29, C31, C32, C33, C34, C35, C36, C37, C38, C39, C40, C41: LCSC Part (none) -> C162422
- C30: LCSC Part (none) -> C162422; LCSC Part# C2168216 -> C162422
- C49, C58, C59, C60, C61: LCSC Part (none) -> C106248
- C55, C56: footprint core:C_0603 -> Capacitor_SMD:C_1210_3225Metric; LCSC Part (none) -> C77101
- C57: LCSC Part (none) -> C29936
- R12: LCSC Part (none) -> C54102347
- R13: LCSC Part (none) -> C2907009
- R14: LCSC Part (none) -> C2906974
- R15, R59: LCSC Part (none) -> C98220
- R24: footprint core:R0603 -> core:R_0603; LCSC Part (none) -> C98220
- R42: value 100k -> 100k 0.5%; LCSC Part (none) -> C122538
- R43: value 19.1k -> 19.1k 0.5%; LCSC Part (none) -> C861184
- R44: LCSC Part (none) -> C2906980
- R45: value 40k -> 40.2k; LCSC Part (none) -> C286588
- R47, R48, R55, R56, R57, R58: LCSC Part (none) -> C14676
- R49: LCSC Part (none) -> C73811
- R54: LCSC Part (none) -> C2907044
Connections:
- net PGND is gone; now on net GND: C21.2, C22.2, C25.2, C26.2, C27.2, C28.2, C29.2, C30.2, C31.2, C32.2, C33.2, C34.2, C35.2, C36.2, C37.2, C38.2, C39.2, C40.2, C41.2, C49.2, C50.1, C52.1, C53.1, C54.1, C55.1, C56.1, C58.1, C59.2, C60.2, C61.2, D11.2 (A), J9.1 (-), LED1.1 (K), LED2.1 (K), LED3.1 (K), LED6.1 (K), R1.1, R13.1, R2.1, R24.1, R3.1, R43.1, R45.1, U3.10 (SNA), U3.11 (SNB), U3.20 (SNC), U3.40 (PGND), U3.41 (EP), U6.1 (GND), U7.4 (GND), U8.2 (GND)
- net at R55.1: now also J8.1
- net at R56.1: now also J8.2
- net at R57.1: now also J8.3
- net at R58.1: now also J8.4
Other:
- note removed: "25V rated"
- note removed: "NET TIE"
- note removed: "This is used for Layout mostly as a ref"
- moved on the sheet: C49, C50, C51, C52, C53, C54, C55, C56, C57, C58, C59, C60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

Commit message: Completed ESC PCB
Parts:
- removed J9: XT30PW-M, my_connector:CONN-TH_XT30PW-M, symbol connector:XT30PW-M
- removed TP1, TP2, TP3, TP4: (no value), TestPoint:TestPoint_Pad_D1.5mm, symbol connector:TestPoint
- added J11: XT30PW-M, my_connector:CONN-TH_XT30PW-M, symbol my_connector:XT30PW-M
- added J12: (no value), my_connector:3x3BusBar Pad, symbol my_connector:BusBar_Pad
- added J9: (no value), my_connector:5x3BusBar Pad, symbol my_connector:BusBar_Pad
Connections:
- net GND: now also J11.1 (-)
- net PWR_IN: now also J11.2 (+)
- net VBUS: now also J12.1, J9.1
Other:
- note added: "Bus bar pad for higher currents"
