File: electrical/mec-arm-esc/peripherals.kicad_sch (KiCad schematic)
At the start: 9 parts, among them U1 TCAN330DCNT

Commit message: Added peripheral systems, and corresponding mcu entries
Parts:
- added C42: 0.1uF, symbol Device:C
- added C43: 1nF, symbol Device:C
- added C44, C45: 100nF, symbol Device:C
- added C46, C47, C48: 10pF, symbol Device:C
- added D1, D2, D3, D4, D5: BAT30KFILM, core:SOD-523_L1.2-W0.8-LS1.6-RD-1, symbol core:BAT30KFILM
- added DA2: USBLC6-2P6, core:SOT-666-6_L1.6-W1.2-P0.50-LS1.6-BR, symbol core:USBLC6-2P6
- added J1: GT-A1257WRS-103SBT01, connector:CONN-SMD_GT-A1257WRS-103SBT01, symbol connector:GT-A1257WRS-103SBT01
- added J2: BM04B-GHS-TBT, connector:CONN-SMD_4P-P1.25_BM04B-GHS-TBT-LF-SN, symbol connector:BM04B-GHS-TBT
- added J3: SM05B-GHS-TB, connector:CONN-SMD_5P-P1.25_SM05B-GHS-TB-LF-SN, symbol connector:SM05B-GHS-TB
- added R22: 120, symbol Device:R
- added R23: 1M, symbol Device:R
- added R24, R25, R26: 0, symbol Device:R
- added R27, R28, R29, R30, R31, R32: 1.8k, symbol Device:R
- added R33: 100k, symbol Device:R
- added R34: 6.38k, symbol Device:R
- added R35: 10.24k, symbol Device:R
- added R4: 10k, core:R0603, symbol core:ERT-J1VG103FA
- added U4: ESD2CAN24DBZRQ1, core:SOT-23-3_L2.9-W1.3-P1.90-LS2.4-BR, symbol core:ESD2CAN24DBZRQ1
- added U5: AS5047P-ATSM_C22459881, core:TSSOP-14_L5.0-W4.4-P0.65-LS6.4-BL, symbol core:AS5047P-ATSM_C22459881
Connections:
- net GND: now also U1.2 (GND), U1.5 (SHDN), U1.8 (S), C42.2, C43.1, C44.2, C45.1, C46.2, C47.2, C48.2, DA2.2 (GND), J1.1, J2.1, J3.1, R23.1, R34.1, R35.1, U4.3 (GND), U5.13 (GND), U5.5 (Test)
- net at USB1.SH (SHIELD): now also C43.2, R23.2
- net FDCAN_TX: now reaches U1.1 (TXD)
- net +3V3: now reaches U1.3 (VCC)
- net +3V3: now also C42.1, C44.1, D1.1 (K), D2.1 (K), D3.1 (K), D4.1 (K), R30.2, R31.2, R32.2, R4.2, U5.11 (VDD), U5.12 (VDD3V3)
- net FDCAN_RX: now reaches U1.4 (RXD)
- net at U1.6 (CANL): now also J1.3, R22.1, U4.2 (IO)
- net at U1.7 (CANH): now also J1.2, R22.2, U4.1 (IO)
- new net: DA2.3 (I/O2), J2.2
- new net: DA2.1 (I/O1), J2.3
- new net +5V_ESC: C45.2, DA2.5 (VBUS), J2.4, J3.2
- new net ENC_A: C48.1, D3.2 (A), J3.3, R26.2, R29.1, R29.2, R32.1
- new net ENC_B: C47.1, D2.2 (A), J3.4, R25.2, R28.1, R28.2, R31.1
- new net ENC_Z: C46.1, D1.2 (A), J3.5, R24.2, R27.1, R27.2, R30.1
- new net MAG_A: R26.1, U5.7 (A)
- new net MAG_B: R25.1, U5.6 (B)
- new net MAG_Z: R24.1, U5.14 (I/PWM)
- new net SPI_ENC_CS: U5.1 (CSn)
- new net SPI_MISO: U5.3 (MISO)
- new net SPI_MOSI: U5.4 (MOSI)
- new net SPI_SCK: U5.2 (CLK)
- new net TEMP_SENSE: D5.2 (A), R35.2, R4.1
- new net UART_RX: DA2.6 (I/O1)
- new net UART_TX: DA2.4 (I/O2)
- new net VBUS: R33.2
- new net VBUS_SENSE: D4.2 (A), R33.1, R34.2
- no-connect marks 3 -> 11
Other:
- note added: "10k at 25, 3380K"
- note added: "CAN"
- note added: "CAN Connector"
- note added: "ENCODERS"
- note added: "Encoder A, B signal input to shift down a 5V encoders signal. Both the internal and external encoders share the same filter. This was done for 3 main reasons: 1. Prevent adding additional circuitry to prevent 3V3 pullup 2. Have some protection in way of MCU 3. (personal pref) Connector can be used for encoder pin debug"
- note added: "External Encoder"
- note added: "Magnetic Encoder"
- note added: "Magnetic Encoder is onboard, and is used when the esc is mounted behind a motor to read absolute position of the motor. It also provides A, B, and Z Signals, but absolute position will likely be preffered over these signals. However, there is the option of using an external encoder, in which case the user !!MUST REMOVE THE RESISTORS CONNECTING TO THE ENCODER!! Both an external and internal encode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"
- note added: "TEMP SENSING"
- note added: "This NTC resistors is 10k at 25 degrees. At 100 degrees, with B = 3380K, they are 1.024k. The max temp which may be read is 100 degrees. 100 degrees = 3V 25 degrees = 1.67V"
- note added: "This maps a voltage range from 50V to 0, where 50V = 3V"
- note added: "UART"
- note added: "UART Connector"
- note added: "USB"
- note added: "VBUS SENSING"
- note removed: "Tie through ESD diode"
- moved on the sheet: DA1, R16, R17, R18, R19, R20, R21, U1, USB1

Commit message: Schematic Done, review 1
Parts:
- added D6, D7, D8, D9: BAT30KFILM, core:SOD-523_L1.2-W0.8-LS1.6-RD-1, symbol core:BAT30KFILM
- added J3: S8B-PHDSS, connector:CONN-TH_S8B-PHDSS-LF-SN, symbol connector:S8B-PHDSS
- added J4, J5: XY-SM02B-GHS-TB, connector:CONN-SMD_SM02B-GHS-TB-LF-SN, symbol connector:XY-SM02B-GHS-TB
- added J6: Conn_02x03_Counter_Clockwise_MountingPin, Connector_PinHeader_2.54mm:PinHeader_2x03_P2.54mm_Vertical, symbol Connector_Generic_MountingPin:Conn_02x03_Counter_Clockwise_MountingPin
- added J7: Conn_02x01, Connector_PinHeader_2.54mm:PinHeader_1x02_P2.54mm_Vertical, symbol Connector_Generic:Conn_02x01
- added LED4, LED5: LTST-C171KGKT, core:LED0805-RD, symbol core:LTST-C171KGKT
- added Q7, Q8: PJA138K_R1_00001, core:SOT-23_L2.9-W1.3-P1.90-LS2.4-BR, symbol core:PJA138K_R1_00001
- added R36, R37, R38, R39, R40, R41, R50, R51, R52, R53, R60, R61: 1k, symbol Device:R
Connections:
- net +3V3: now also D6.1 (K), D7.1 (K), D8.1 (K), D9.1 (K), J6.5 (Pin_5)
- net +5V_ESC: now also J3.2, J4.1, J5.1
- net GND: now also J3.1, J6.1 (Pin_1), J7.1 (Pin_1), LED4.1 (K), LED5.1 (K), Q7.2 (S), Q8.2 (S), R60.2, R61.2
- new net: LED4.2 (A), R50.1
- new net: LED5.2 (A), R51.1
- new net: Q8.1 (G), R53.1, R61.1
- new net: Q7.1 (G), R52.1, R60.1
- new net: J4.2, Q7.3 (D)
- new net: J5.2, Q8.3 (D)
- new net ADC_FORCE1+: D7.2 (A), R36.1
- new net ADC_FORCE1-: D9.2 (A), R39.2
- new net ADC_FORCE2+: D6.2 (A), R37.1
- new net ADC_FORCE2-: D8.2 (A), R38.2
- new net DAC_OUT1: J7.2 (Pin_2)
- new net EXT_FORCE1+: J3.6, R36.2
- new net EXT_FORCE1-: J3.5, R39.1
- new net EXT_FORCE2+: J3.8, R37.2
- new net EXT_FORCE2-: J3.7, R38.1
- new net FAN_CTRL: R53.2
- new net GPIO_CTRL1: J3.4, R40.2
- new net GPIO_CTRL2: J3.3, R41.1
- new net GPIO_EXT1: R40.1
- new net GPIO_EXT2: R41.2
- new net LASER_CTRL: R52.2
- new net LED_DEBUG1: R50.2, R51.2
- new net NRST: J6.2 (Pin_2)
- new net SWCLK: J6.4 (Pin_4)
- new net SWDIO: J6.6 (Pin_6)
- no-connect marks 11 -> 17
Other:
- note added: "COMMUNICATION"
- note added: "DEBUG"
- note added: "External Env Sensing"
- note added: "FAN AND LAZER CONTROL"
- note added: "FLASHING"
- note added: "MCU SENSING"
- note added: "Setup here is mostly for if we have any type of sensing (strain gauge or haptic sensing) that is a passive board."
- moved on the sheet: C42, C43, C44, C45, C46, C47, C48, DA1, DA2, J1, J2, J3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

Commit message: Done placement, starting routing
Parts:
- removed J3: S8B-PHDSS, connector:CONN-TH_S8B-PHDSS-LF-SN, symbol connector:S8B-PHDSS
- removed J4, J5: XY-SM02B-GHS-TB, connector:CONN-SMD_SM02B-GHS-TB-LF-SN, symbol connector:XY-SM02B-GHS-TB
- removed J6: Conn_02x03_Counter_Clockwise_MountingPin, Connector_PinHeader_2.54mm:PinHeader_2x03_P2.54mm_Vertical, symbol Connector_Generic_MountingPin:Conn_02x03_Counter_Clockwise_MountingPin
- removed Q7: PJA138K_R1_00001, core:SOT-23_L2.9-W1.3-P1.90-LS2.4-BR, symbol core:PJA138K_R1_00001
- removed R24, R25, R26: 0, symbol Device:R
- removed R60: 1k, symbol Device:R
- removed USB1: USB4215-03-A, connector:USB-C-SMD_GT-USB-7010B, symbol connector:USB_C_Receptacle_USB2.0_16P
- added J4: S10B-PHDSS, my_connector:CONN-TH_S10B-PHDSS-LF-SN, symbol my_connector:S10B-PHDSS
- added J5: XY-SM02B-GHS-TB, my_connector:CONN-SMD_SM02B-GHS-TB-LF-SN, symbol my_connector:XY-SM02B-GHS-TB
- added J6: Header_2Rows-05Pins, my_connector:PinHeader_2_row_5_pin_P2.54mm_Vertical, symbol my_connector:Header_2Rows-05Pins
- added JP1, JP2, JP3, JP4: SolderJumper_2_Open, Jumper:SolderJumper-2_P1.3mm_Open_TrianglePad1.0x1.5mm, symbol connector:SolderJumper_2_Open
- added R46: 1k, core:R_0603, symbol Device:R
- added USB1: USB4215-03-A, my_connector:USB-C-SMD_GT-USB-7010B, symbol my_connector:USB4215-03-A
- C42, C43, C44, C45, C46, C47, C48: footprint (none) -> core:C_0603
- J1: footprint connector:CONN-SMD_GT-A1257WRS-103SBT01 -> my_connector:CONN-SMD_GT-A1257WRS-103SBT01
- J2: footprint connector:CONN-SMD_4P-P1.25_BM04B-GHS-TBT-LF-SN -> my_connector:CONN-SMD_4P-P1.25_BM04B-GHS-TBT-LF-SN
- J3: footprint connector:CONN-SMD_5P-P1.25_SM05B-GHS-TB-LF-SN -> my_connector:CONN-SMD_5P-P1.25_SM05B-GHS-TB-LF-SN
- R16, R17, R18, R19, R20, R21, R23, R27, R28, R29, R30, R31, R32, R33, R34, R35, R36, R37, R38, R39, R40, R41, R50, R51, R52, R53, R61: footprint (none) -> core:R_0603
- R22: footprint (none) -> core:R_0603; now fitted
Connections:
- net +3V3: now also D5.1 (K), J6.5 (Pin_5)
- net +5V_ESC: now also J4.2
- net +5V_USB: now also USB1.A4B9 (VBUS), USB1.B4A9 (VBUS)
- net ENC_A: now also C46.1, D1.2 (A), J3.5, R27.1, R27.2, R30.1, JP4.1 (A); no longer C48.1, D3.2 (A), J3.3, R29.1, R29.2, R32.1
- net ENC_B: now also JP3.1 (A)
- net ENC_Z: now also C48.1, D3.2 (A), J3.3, R29.1, R29.2, R32.1, JP2.1 (A); no longer C46.1, D1.2 (A), J3.5, R27.1, R27.2, R30.1
- net EXT_FORCE1+: now also J4.8
- net EXT_FORCE1-: now also J4.7
- net EXT_FORCE2+: now also J4.10
- net EXT_FORCE2-: now also J4.9
- net GND: now also J6.1 (Pin_1), USB1.A1B12 (GND), USB1.B1A12 (GND); no longer Q8.2 (S), R34.1
- net GPIO_CTRL1: now also J4.6
- net GPIO_CTRL2: now also J4.5
- net LASER_CTRL: now also R46.1; no longer R52.2
- net MAG_A: now also JP4.2 (B)
- net MAG_B: now also JP3.2 (B)
- net MAG_Z: now also JP2.2 (B)
- net NRST: now also J6.3 (Pin_3)
- net SWCLK: now also J6.2 (Pin_2)
- net SWDIO: now also J6.4 (Pin_4)
- net VBUS: now also J5.1
- net USB_D_N: now reaches DA1.1 (I/O1)
- net USB_D_N: now also USB1.A7 (Dn1), USB1.B7 (Dn2)
- net USB_D_P: now reaches DA1.3 (I/O2)
- net USB_D_P: now also USB1.A6 (Dp1), USB1.B6 (Dp2)
- net UART_TX_OUT: now reaches DA2.3 (I/O2), J2.2
- net UART_RX_OUT: now reaches DA2.1 (I/O1), J2.3
- net at C43.2, R23.2: now also USB1.13 (EH), USB1.14 (EH), USB1.15 (EH), USB1.16 (EH)
- net at R18.1: now also USB1.B5 (CC2)
- net CAN_P: now reaches J1.2, R22.2, U1.7 (CANH)
- net CAN_P: now also U4.2 (IO); no longer U4.1 (IO)
- net CAN_N: now reaches J1.3, U1.6 (CANL)
- net CAN_N: now also U4.1 (IO), JP1.2 (B); no longer R22.1, U4.2 (IO)
- net at R52.1: now also J4.3
- net at Q8.3 (D): now also J5.2
- net at R19.1: now also USB1.A5 (CC1)
- new net: JP1.1 (A), R22.1
- new net GPIO_EXT3: R52.2
- new net LASER: J4.4, R46.2
- new net PGND: J4.1, Q8.2 (S), R34.1
- no-connect marks 17 -> 13
Other:
- note added: "FAN CONTROL"
- note removed: "FAN AND LAZER CONTROL"
- moved on the sheet: C43, J1, J7, LED4, LED5, Q8, R23, R50, R51, R53, R61, U4

Commit message: All signal routing finishes, power and planes not yet
Parts:
- removed D6, D7, D8, D9: BAT30KFILM, core:SOD-523_L1.2-W0.8-LS1.6-RD-1, symbol core:BAT30KFILM
- removed LED4: LTST-C171KGKT, core:LED0805-RD, symbol core:LTST-C171KGKT
- added C62: 0.1uF, core:C_0603, symbol Device:C
- added JP5: SolderJumper_2_Open, Jumper:SolderJumper-2_P1.3mm_Open_TrianglePad1.0x1.5mm, symbol connector:SolderJumper_2_Open
- added R60, R68, R69: 1k, core:R_0603, symbol Device:R
- added R70, R71, R72: 1.8k, core:R_0603, symbol Device:R
- C42, C44, C45: LCSC Part (none) -> C108079
- C43: value 1nF -> 10nF; LCSC Part (none) -> C519406
- C46, C47, C48: LCSC Part (none) -> C2168592
- J6, J7: now not fitted
- R16, R17: LCSC Part (none) -> C844919
- R18, R19: LCSC Part (none) -> C2907044
- R20, R21, R33: LCSC Part (none) -> C2906980
- R22: LCSC Part (none) -> C2906988
- R23: value 1M -> 2.55M; LCSC Part (none) -> C54102347
- R27, R28, R29, R30, R31, R32: LCSC Part (none) -> C286575
- R34: value 6.38k -> 6.34k; LCSC Part (none) -> C321969
- R35: value 10.24k -> 3.24k; LCSC Part (none) -> C728589
- R36, R37, R38, R39, R40, R41, R46, R50, R51, R52, R53, R61: LCSC Part (none) -> C14676
Connections:
- net PGND is gone; now on net GND: J4.1, Q8.2 (S), R34.1
- net +3V3: now also DA2.5 (VBUS), J4.2, C62.2
- net +5V_ESC: now also JP5.2 (B); no longer DA2.5 (VBUS), J2.4, J4.2
- net CAN_N: now also R22.1; no longer JP1.2 (B)
- net CAN_P: now also JP1.2 (B); no longer R22.2
- net DAC_OUT1: now also R60.2; no longer J7.2 (Pin_2)
- net ENC_A: now also R70.1; no longer J3.5, JP4.1 (A), R27.1
- net ENC_B: now also R71.1; no longer J3.4, JP3.1 (A), R28.1
- net ENC_Z: now also R72.1; no longer J3.3, JP2.1 (A), R29.1
- net GND: now also R50.1, C62.1
- net GPIO_CTRL1: now also J4.5, R41.1; no longer J4.6, R40.2
- net GPIO_CTRL2: now also J4.6, R40.2; no longer J4.5, R41.1
- net GPIO_EXT1: now also R41.2; no longer R40.1
- net GPIO_EXT2: now also R40.1; no longer R41.2
- net LASER_CTRL: now also R50.2
- net LED_DEBUG1: no longer R50.2
- net UART_RX: now also R68.1; no longer DA2.6 (I/O1)
- net UART_TX: now also R69.1; no longer DA2.4 (I/O2)
- net USB_D_O_P: now reaches DA1.4 (I/O2), R17.2
- net USB_D_O_N: now reaches DA1.6 (I/O1), R16.2
- net at JP1.1 (A): now also R22.2; no longer R22.1
- net ADC_FORCE1+ renamed ADC_FORCE1
- net ADC_FORCE1- renamed ADC_FORCE2
- net ADC_FORCE2+ renamed ADC_FORCE3
- net ADC_FORCE2- renamed ADC_FORCE4
- net EXT_FORCE1+ renamed EXT_FORCE1
- net EXT_FORCE1- renamed EXT_FORCE2
- net EXT_FORCE2+ renamed EXT_FORCE3
- net EXT_FORCE2- renamed EXT_FORCE4
- new net: J2.4, JP5.1 (A)
- new net: JP4.1 (A), R70.2
- new net: DA2.4 (I/O2), R69.2
- new net: DA2.6 (I/O1), R68.2
- new net: J7.2 (Pin_2), R60.1
- new net: JP2.1 (A), R72.2
- new net: JP3.1 (A), R71.2
- new net ENC_A_IN: J3.5, R27.1
- new net ENC_B_IN: J3.4, R28.1
- new net ENC_Z_IN: J3.3, R29.1
Other:
- note added: "This NTC resistors is 10k at 25 degrees. At 100 degrees, with B = 3380K, they are 1.024k. The max temp which may be read safely is 150 degrees. 150 degrees = 3V 25 degrees = 0.82V"
- note added: "This UART connector is used for either debug, or to power and communicate with another device. Thus, a bridge is needed so in the sebug case, 5V is nor provided"
- note removed: "This NTC resistors is 10k at 25 degrees. At 100 degrees, with B = 3380K, they are 1.024k. The max temp which may be read is 100 degrees. 100 degrees = 3V 25 degrees = 1.67V"
- moved on the sheet: J4, JP2, JP3, LED5, R22, R27, R28, R29, R36, R37, R38, R39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

Commit message: Completed ESC PCB
Parts:
- removed JP2: SolderJumper_2_Open, Jumper:SolderJumper-2_P1.3mm_Open_TrianglePad1.0x1.5mm, symbol connector:SolderJumper_2_Open
- removed R72: 1.8k, core:R_0603, symbol Device:R
- J2, J4: now not fitted
Connections:
- net +3V3: no longer C62.2, DA2.5 (VBUS)
- net +5V_ESC: now also C62.2, DA2.5 (VBUS)
- net ENC_A: now also R71.1; no longer R70.1
- net ENC_B: now also R70.1; no longer R71.1
- net MAG_A: now also JP3.2 (B); no longer JP4.2 (B)
- net MAG_B: now also JP4.2 (B); no longer JP3.2 (B)
- net MAG_Z: no longer names the net of U5.14 (I/PWM)
- no-connect marks 13 -> 14
